File: PCB/PCB.kicad_pcb (KiCad board)
At the start: 2 copper layers, 26 parts, among them J1 HC-SR04 Breakout, J2 Conn_01x06_Socket, SW1 RST, SW2 BOOT, SW3 SW_SPDT, U1 MQ-2 Sensor, U2 ESP32-WROOM-32, U3 DHT22, U4 MPU-6050, U5 AMS1117-3.3

Commit message: [ADDED] PCB Design Completed
Parts:
- added ?: , , F.Cu at (231.4, 117.7)
- added ?: , , F.Cu at (231.0, 71.3)
- added ?: , , F.Cu at (171.9, 117.6)
- added BZ1: Buzzer, Buzzer_Beeper:Buzzer_D14mm_H7mm_P10mm, F.Cu at (199.5, 101.2)
- added G***: LOGO, LOGO, F.Cu at (171.7, 106.7)
- added G***: LOGO, LOGO, F.Cu at (203.6, 125.5)
- added J3: Battery, Connector_JST:JST_EH_S2B-EH_1x02_P2.50mm_Horizontal, F.Cu at (175.4, 94.0)
- C1, C2, C3, C4, C5, C6, C7, C8, C9: footprint Capacitor_SMD:C_0805_2012Metric -> Capacitor_SMD:C_0603_1608Metric
- R1, R2, R3, R4, R5, R6, R7: footprint Resistor_THT:R_Axial_DIN0207_L6.3mm_D2.5mm_P10.16mm_Horizontal -> Resistor_SMD:R_0603_1608Metric
- SW3: footprint Button_Switch_THT:SW_Slide_SPDT_Straight_CK_OS102011MS2Q -> Button_Switch_THT:SW_Slide_SPDT_Angled_CK_OS102011MA1Q
- U3: footprint Sensor:Aosong_DHT11_5.5x12.0_P2.54mm -> custom:DHT22_Horizontal
- moved U1 142.8 mm to (222.0, 109.2)
- moved J2 134.3 mm to (227.3, 81.0)
- moved C4 121.9 mm to (228.6, 74.2), turned to -90 degrees
- moved C5 119.8 mm to (225.2, 74.2), turned to 90 degrees
- moved C8 117.3 mm to (226.9, 74.2), turned to 90 degrees
- moved U4 117.0 mm to (221.4, 73.7), turned to 90 degrees
- moved C6 115.6 mm to (217.2, 70.0), turned to 90 degrees
- moved SW2 113.1 mm to (216.7, 91.0), turned to 180 degrees
- moved U2 107.8 mm to (204.7, 77.9)
- moved J1 104.8 mm to (221.6, 81.2)
- moved R3 97.6 mm to (222.7, 97.0), turned to -90 degrees
- moved C2 96.4 mm to (193.1, 71.0), turned to 180 degrees
- moved SW1 94.4 mm to (187.9, 71.8)
- moved R7 93.8 mm to (217.2, 76.5), turned to 90 degrees
- moved R6 93.6 mm to (217.2, 73.2), turned to -90 degrees
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Connections:
- U2 pad 16: unconnected-(U2-IO13-Pad16) -> /BUZZER
- U2 pad 23: unconnected-(U2-IO15-Pad23) -> /DHT22
- U2 pad 27: /DHT22 -> /TRIG
- U2 pad 29: /TRIG -> unconnected-(U2-IO5-Pad29)
- U2 pad 33: unconnected-(U2-IO21-Pad33) -> /SDA
- U2 pad 36: unconnected-(U2-IO22-Pad36) -> /SCL
Routing:
- net GND: track 0.00 -> 208.1 mm, vias 0 -> 8
- net /VDD33: track 0.00 -> 159.3 mm, vias 0 -> 12
- net /VIN_BATT: track 0.00 -> 93.6 mm, vias 0 -> 1
- net /MQ2_OUT: track 0.00 -> 70.8 mm, vias 0 -> 1
- net /EN: track 0.00 -> 61.8 mm, vias 0 -> 1
- net /DHT22: track 0.00 -> 42.9 mm
- net /MPU_INTER: track 0.00 -> 39.9 mm, vias 0 -> 2
- net /BATT OUT: track 0.00 -> 23.1 mm
- net /RXD0: track 0.00 -> 22.9 mm, vias 0 -> 1
- net /IO0: track 0.00 -> 22.5 mm
- net /TXD0: track 0.00 -> 21.3 mm, vias 0 -> 1
- net /BUZZER: track 0.00 -> 14.0 mm
- net /V_IND: track 0.00 -> 10.4 mm
- net /ECHO: track 0.00 -> 8.76 mm
- net /TRIG: track 0.00 -> 8.23 mm
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- added copper zone on F.Cu, net /VIN_BATT
- added copper zone on F.Cu, net GND
- added copper zone on In1.Cu, net GND
- added copper zone on In2.Cu, net GND
Other:
- board outline added: 66.8 x 59.2 mm
- copper layers 2 -> 4
- board text added: "BUZZER"
- board text added: "DHT22"
- board text added: "MQ-2"
- board text added: "cc@edgecutterr"
