File: PCB/PCB.kicad_sch (KiCad schematic)
At the start: 0 parts

Commit message: Ignore KiCad auto-generated history files
Parts:
- added C1, C4, C6: 0.1uF, symbol Device:C
- added C2: C, symbol Device:C
- added C3: 10uF, symbol Device:C
- added C5: 0.01uF, symbol Device:C
- added C7: 2.2nF, symbol Device:C
- added C8: 2.2uF, symbol Device:C
- added C9: 1uF, symbol Device:C
- added J1: Conn_01x06_Socket, symbol Connector:Conn_01x06_Socket
- added R1: 2.2 kΩ, symbol Device:R_Small_US
- added R2: 2.2 KΩ, symbol Device:R_Small_US
- added R3, R4: 10 kΩ, symbol Device:R_US
- added SW1: RST, symbol Switch:SW_Push
- added SW2: BOOT, symbol Switch:SW_Push
- added SW3: SW_SPDT, symbol Switch:SW_SPDT
- added U1: ESP32-WROOM-32, RF_Module:ESP32-WROOM-32, symbol RF_Module:ESP32-WROOM-32
- added U2: AMS1117-3.3, Package_TO_SOT_SMD:SOT-223-3_TabPin2, symbol Regulator_Linear:AMS1117-3.3
- added U3: MPU-6050, Sensor_Motion:InvenSense_QFN-24_4x4mm_P0.5mm, symbol Sensor_Motion:MPU-6050
Connections:
- new net: C6.1, U3.10 (REGOUT)
- new net: C7.1, U3.20 (CPOUT)
- new net: C2.1, SW3.1 (A), U2.3 (VI)
- new net BATT OUT: SW3.2 (B)
- new net EN: C9.1, J1.3 (Pin_3), R3.1, SW1.2, U1.3 (EN)
- new net GND: C1.2, C2.2, C3.2, C4.2, C5.2, C6.2, C7.2, C8.2, C9.2, J1.6 (Pin_6), SW1.1, SW2.2, U1.1 (GND), U1.15 (GND), U1.38 (GND), U1.39 (GND), U2.1 (GND), U3.1 (CLKIN), U3.11 (FSYNC), U3.18 (GND), U3.9 (AD0)
- new net IO0: J1.4 (Pin_4), R4.1, SW2.1, U1.25 (IO0)
- new net MPU_INTER: U3.12 (INT)
- new net RXD0: J1.2 (Pin_2), U1.34 (RXD0/IO3)
- new net SCL: R2.2, U3.23 (SCL)
- new net SDA: R1.2, U3.24 (SDA)
- new net TXD0: J1.1 (Pin_1), U1.35 (TXD0/IO1)
- new net VDD33: C1.1, C3.1, C4.1, C5.1, C8.1, J1.5 (Pin_5), R1.1, R2.1, R3.2, R4.2, U1.2 (VDD), U2.2 (VO), U3.13 (VDD), U3.8 (VLOGIC)
- no-connect marks 0 -> 12
Other:
- note added: "MPU 6050"
- note added: "Programming Headders"
- note added: "Voltage Regulator"
- company: (none) -> Rohit Patki
- title: (none) -> Miners Safety Helmet

Commit message: [ADDED] Sensors and Footprints Assignments
 - Added sensors like mq 2 dht 22 and hcsr 04
-  Assigned footprints for registration capacitors with  1608 metric sizes
- Created custom footprint and symbol for MQ2 sensor
Parts:
- added J1: HC-SR04 Breakout, Connector_PinSocket_2.54mm:PinSocket_1x04_P2.54mm_Vertical, symbol Connector:Conn_01x04_Socket
- added R1, R2: 1k Ω, Resistor_SMD:R_0603_1608Metric, symbol Device:R_US
- added R3: 3.3 kΩ, Resistor_SMD:R_0603_1608Metric, symbol Device:R_US
- added U1: MQ-2 Sensor, custom:MQ2, symbol Miners:MQ-3
- added U3: DHT22, Sensor:Aosong_DHT11_5.5x12.0_P2.54mm, symbol Sensor:DHT11
- C1: renamed from C9; footprint (none) -> Capacitor_SMD:C_0603_1608Metric
- C2: renamed from C1; footprint (none) -> Capacitor_SMD:C_0603_1608Metric
- C3: renamed from C2; footprint (none) -> Capacitor_SMD:C_0603_1608Metric
- C4: renamed from C6; footprint (none) -> Capacitor_SMD:C_0603_1608Metric
- C5, C8: footprint (none) -> Capacitor_SMD:C_0603_1608Metric
- C6: renamed from C7; footprint (none) -> Capacitor_SMD:C_0603_1608Metric
- C7: renamed from C3; footprint (none) -> Capacitor_SMD:C_0603_1608Metric
- C9: renamed from C4; footprint (none) -> Capacitor_SMD:C_0603_1608Metric
- J2: renamed from J1; footprint (none) -> Connector_PinSocket_2.54mm:PinSocket_1x06_P2.54mm_Vertical
- R4: renamed from R3; footprint (none) -> Resistor_SMD:R_0603_1608Metric
- R5: renamed from R4; footprint (none) -> Resistor_SMD:R_0603_1608Metric
- R6: renamed from R2; footprint (none) -> Resistor_SMD:R_0603_1608Metric
- R7: renamed from R1; footprint (none) -> Resistor_SMD:R_0603_1608Metric
- SW1, SW2: footprint (none) -> Button_Switch_SMD:SW_Push_1P1T_NO_CK_KMR2
- SW3: footprint (none) -> Button_Switch_THT:SW_Slide_SPDT_Straight_CK_OS102011MS2Q
- renumbered U1 to U2, U3 to U4, U2 to U5
Connections:
- net GND: now also J1.4 (Pin_4), R2.2, R3.1, U1.5 (H2), U3.4 (GND)
- net MPU_INTER: now also U2.13 (IO14)
- net VDD33: now also U3.1 (VDD)
- net ECHO: now reaches U2.26 (IO4)
- net ECHO: now also J1.3 (Pin_3)
- net DHT22: now reaches U2.27 (IO16)
- net DHT22: now also U3.2 (DATA)
- net TRIG: now reaches U2.29 (IO5)
- net TRIG: now also J1.2 (Pin_2)
- net V_IND: now reaches U2.6 (IO34)
- net V_IND: now also R1.2, R2.1
- net MQ2_OUT: now reaches U2.8 (IO32)
- net MQ2_OUT: now also R3.2, U1.4 (B1), U1.6 (B2)
- net VIN_BATT: now reaches C3.1, SW3.1 (A), U5.3 (VI)
- net VIN_BATT: now also J1.1 (Pin_1), R1.1, U1.1 (A1), U1.2 (H1), U1.3 (A2)
- no-connect marks 12 -> 26
Other:
- note added: "BATT-IND"
- note added: "DHT22"
- note added: "ESP32-Wroom-32 Module"
- note added: "HC-SR04 Breakout"
- note added: "MQ-2 Sensor"
- moved on the sheet: C1, C2, J2, R4, R5, SW1, SW2, U2

Commit message: [ADDED] PCB Design Completed
Parts:
- added BZ1: Buzzer, Buzzer_Beeper:Buzzer_D14mm_H7mm_P10mm, symbol Device:Buzzer
- added J3: Battery, Connector_JST:JST_EH_S2B-EH_1x02_P2.50mm_Horizontal, symbol Connector:Conn_01x02_Socket
- SW3: footprint Button_Switch_THT:SW_Slide_SPDT_Straight_CK_OS102011MS2Q -> Button_Switch_THT:SW_Slide_SPDT_Angled_CK_OS102011MA1Q
- U3: footprint Sensor:Aosong_DHT11_5.5x12.0_P2.54mm -> custom:DHT22_Horizontal
Connections:
- net BATT OUT: now also J3.1 (Pin_1)
- net DHT22: now also U2.23 (IO15); no longer U2.27 (IO16)
- net GND: now also BZ1.2 (-), J3.2 (Pin_2)
- net SCL: now also U2.36 (IO22)
- net SDA: now also U2.33 (IO21)
- net TRIG: now also U2.27 (IO16); no longer U2.29 (IO5)
- net BUZZER: now reaches U2.16 (IO13)
- net BUZZER: now also BZ1.1 (+)
- no-connect marks 26 -> 22
Other:
- note added: "BATT CONN"
- note added: "BUZZER"
